File: KiCad/Drawer_Controller/Drawer_Controller/VDD_Switch.kicad_sch (KiCad schematic)
At the start: 6 parts, among them Q3 AO3400A, Q4 AO3401A

Commit message: More progress
Parts:
- removed D2: MBRS340, MBRS340:DIOM7959X261N, symbol MBRS340:MBRS340
- R10, R11, R12: footprint (none) -> Resistor_SMD:R_0805_2012Metric_Pad1.20x1.40mm_HandSolder
Changed lines of the file:
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@@
 (kicad_sch (version 20211123) (generator eeschema)
   (paper "A4")
-  (junction (at 142.24 86.36) (diameter 0) (color 0 0 0 0)
-  )
   (junction (at 124.46 78.74) (diameter 0) (color 0 0 0 0)
   )
@@
     (stroke (width 0) (type default) (color 0 0 0 0))
   )
-  (wire (pts (xy 142.24 86.36) (xy 142.24 87.63))
-    (stroke (width 0) (type default) (color 0 0 0 0))
-  )
   (wire (pts (xy 124.46 78.74) (xy 124.46 80.645))
     (stroke (width 0) (type default) (color 0 0 0 0))
@@
   )
   (wire (pts (xy 113.03 85.725) (xy 116.84 85.725))
-    (stroke (width 0) (type default) (color 0 0 0 0))
-  )
-  (wire (pts (xy 142.24 97.79) (xy 142.24 100.33))
     (stroke (width 0) (type default) (color 0 0 0 0))
   )
@@
     (property "Reference" "R10" (id 0) (at 106.045 80.01 90))
     (property "Value" "100" (id 1) (at 106.045 82.55 90))
-    (property "Footprint" "" (id 2) (at 106.045 85.725 0)
+    (property "Footprint" "Resistor_SMD:R_0805_2012Metric_Pad1.20x1.40mm_HandSolder" (id 2) (at 106.045 85.725 0)
       (effects (font (size 1.27 1.27)) hide)
     )
@@
     (pin "1")
   )
-  (symbol (lib_id "MBRS340:MBRS340") (at 142.24 92.71 90)
-    (in_bom yes) (on_board yes)
-    (property "Reference" "D2" (id 0) (at 144.78 91.4399 90)
-      (effects (font (size 1.27 1.27)) (justify right))
-    )
-    (property "Value" "MBRS340" (id 1) (at 144.78 93.9799 90)
-      (effects (font (size 1.27 1.27)) (justify right))
-    )
-    (property "Footprint" "MBRS340:DIOM7959X261N" (id 2) (at 142.24 92.71 0)
-      (effects (font (size 1.27 1.27)) (justify left bottom) hide)
-    )
-    (property "Datasheet" "" (id 3) (at 142.24 92.71 0)
-      (effects (font (size 1.27 1.27)) (justify left bottom) hide)
-    )
-    (property "STANDARD" "IPC-7351B" (id 4) (at 142.24 92.71 0)
-      (effects (font (size 1.27 1.27)) (justify left bottom) hide)
-    )
-    (property "MAXIMUM_PACKAGE_HEIGHT" "2.61mm" (id 5) (at 142.24 92.71 0)
-      (effects (font (size 1.27 1.27)) (justify left bottom) hide)
-    )
-    (property "PARTREV" "14" (id 6) (at 142.24 92.71 0)
-      (effects (font (size 1.27 1.27)) (justify left bottom) hide)
-    )
-    (property "MANUFACTURER" "ON Semiconductor" (id 7) (at 142.24 92.71 0)
-      (effects (font (size 1.27 1.27)) (justify left bottom) hide)
-    )
-    (pin "A")
-    (pin "C")
-  )
   (symbol (lib_id "Device:R_Small") (at 113.03 92.075 0)
     (in_bom yes) (on_board yes) (fields_autoplaced)
@@
       (effects (font (size 1.27 1.27)) (justify left))
     )
-    (property "Footprint" "" (id 2) (at 113.03 92.075 0)
+    (property "Footprint" "Resistor_SMD:R_0805_2012Metric_Pad1.20x1.40mm_HandSolder" (id 2) (at 113.03 92.075 0)
       (effects (font (size 1.27 1.27)) hide)
     )
@@
       (effects (font (size 1.27 1.27)) (justify left))
     )
-    (property "Footprint" "" (id 2) (at 124.46 74.93 0)
+    (property "Footprint" "Resistor_SMD:R_0805_2012Metric_Pad1.20x1.40mm_HandSolder" (id 2) (at 124.46 74.93 0)
       (effects (font (size 1.27 1.27)) hide)
     )
@@
       (effects (font (size 1.27 1.27)) hide)
     )
-    (pin "1")
-  )
-  (symbol (lib_id "power:GND") (at 142.24 100.33 0)
-    (in_bom yes) (on_board yes)
-    (property "Reference" "#PWR0147" (id 0) (at 142.24 106.68 0)
-      (effects (font (size 1.27 1.27)) hide)
-    )
-    (property "Value" "GND" (id 1) (at 142.24 104.14 0))
-    (property "Footprint" "" (id 2) (at 142.24 100.33 0)
-      (effects (font (size 1.27 1.27)) hide)
-    )
-    (property "Datasheet" "" (id 3) (at 142.24 100.33 0)
-      (effects (font (size 1.27 1.27)) hide)
-    )

Commit message: Small adjustments after schematic review with Basti
Changed lines of the file:
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@@
-    (stroke (width 0) (type default) (color 0 0 0 0))
-  )
-  (wire (pts (xy 99.06 91.44) (xy 95.25 91.44))
-    (stroke (width 0) (type default) (color 0 0 0 0))
-  )
-  (wire (pts (xy 95.25 80.01) (xy 99.06 80.01))
     (stroke (width 0) (type default) (color 0 0 0 0))
   )
@@
   )
   (wire (pts (xy 108.585 85.725) (xy 113.03 85.725))
-    (stroke (width 0) (type default) (color 0 0 0 0))
-  )
-  (wire (pts (xy 99.06 93.98) (xy 99.06 91.44))
     (stroke (width 0) (type default) (color 0 0 0 0))
   )
@@
     (stroke (width 0) (type default) (color 0 0 0 0))
   )
-  (wire (pts (xy 99.06 80.01) (xy 99.06 78.105))
-    (stroke (width 0) (type default) (color 0 0 0 0))
-  )
-  (hierarchical_label "+5V" (shape input) (at 95.25 80.01 180)
-    (effects (font (size 1.27 1.27)) (justify right))
-  )
-  (hierarchical_label "GND" (shape input) (at 95.25 91.44 180)
-    (effects (font (size 1.27 1.27)) (justify right))
-  )
   (hierarchical_label "VDD_Switchtable" (shape output) (at 157.48 86.36 0)
     (effects (font (size 1.27 1.27)) (justify left))
@@
   (symbol (lib_id "power:+5V") (at 124.46 71.12 0)
     (in_bom yes) (on_board yes)
-    (property "Reference" "#PWR0142" (id 0) (at 124.46 74.93 0)
+    (property "Reference" "#PWR0115" (id 0) (at 124.46 74.93 0)
       (effects (font (size 1.27 1.27)) hide)
     )
@@
     )
     (property "Datasheet" "" (id 3) (at 124.46 71.12 0)
-      (effects (font (size 1.27 1.27)) hide)
-    )
-    (pin "1")
-  )
-  (symbol (lib_id "power:+5V") (at 99.06 78.105 0)
-    (in_bom yes) (on_board yes)
-    (property "Reference" "#PWR0146" (id 0) (at 99.06 81.915 0)
-      (effects (font (size 1.27 1.27)) hide)
-    )
-    (property "Value" "+5V" (id 1) (at 99.06 74.295 0))
-    (property "Footprint" "" (id 2) (at 99.06 78.105 0)
-      (effects (font (size 1.27 1.27)) hide)
-    )
-    (property "Datasheet" "" (id 3) (at 99.06 78.105 0)
       (effects (font (size 1.27 1.27)) hide)
     )
@@
   (symbol (lib_id "power:+5V") (at 142.24 71.12 0)
     (in_bom yes) (on_board yes)
-    (property "Reference" "#PWR0144" (id 0) (at 142.24 74.93 0)
+    (property "Reference" "#PWR0121" (id 0) (at 142.24 74.93 0)
       (effects (font (size 1.27 1.27)) hide)
     )
@@
   (symbol (lib_id "power:GND") (at 124.46 100.33 0)
     (in_bom yes) (on_board yes)
-    (property "Reference" "#PWR0143" (id 0) (at 124.46 106.68 0)
+    (property "Reference" "#PWR0116" (id 0) (at 124.46 106.68 0)
       (effects (font (size 1.27 1.27)) hide)
     )
@@
     (pin "3")
   )
-  (symbol (lib_id "power:GND") (at 99.06 93.98 0)
-    (in_bom yes) (on_board yes)
-    (property "Reference" "#PWR0145" (id 0) (at 99.06 100.33 0)
-      (effects (font (size 1.27 1.27)) hide)
-    )
-    (property "Value" "GND" (id 1) (at 99.06 97.79 0))
-    (property "Footprint" "" (id 2) (at 99.06 93.98 0)
-      (effects (font (size 1.27 1.27)) hide)
-    )
-    (property "Datasheet" "" (id 3) (at 99.06 93.98 0)
-      (effects (font (size 1.27 1.27)) hide)
-    )
-    (pin "1")
-  )
 )

Commit message: Small progress
Parts:
- renumbered Q3 to Q1, Q4 to Q2, R10 to R7, R11 to R8, R12 to R9
Changed lines of the file:
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@@
   (symbol (lib_id "power:+5V") (at 124.46 71.12 0)
     (in_bom yes) (on_board yes)
-    (property "Reference" "#PWR0115" (id 0) (at 124.46 74.93 0)
+    (property "Reference" "#PWR0136" (id 0) (at 124.46 74.93 0)
       (effects (font (size 1.27 1.27)) hide)
     )
@@
   (symbol (lib_id "Device:R_Small") (at 106.045 85.725 90)
     (in_bom yes) (on_board yes) (fields_autoplaced)
-    (property "Reference" "R10" (id 0) (at 106.045 80.01 90))
+    (property "Reference" "R7" (id 0) (at 106.045 80.01 90))
     (property "Value" "100" (id 1) (at 106.045 82.55 90))
     (property "Footprint" "Resistor_SMD:R_0805_2012Metric_Pad1.20x1.40mm_HandSolder" (id 2) (at 106.045 85.725 0)
@@
   (symbol (lib_id "Transistor_FET:AO3400A") (at 121.92 85.725 0)
     (in_bom yes) (on_board yes) (fields_autoplaced)
-    (property "Reference" "Q3" (id 0) (at 128.27 84.4549 0)
+    (property "Reference" "Q1" (id 0) (at 128.27 84.4549 0)
       (effects (font (size 1.27 1.27)) (justify left))
     )
@@
   (symbol (lib_id "power:+5V") (at 142.24 71.12 0)
     (in_bom yes) (on_board yes)
-    (property "Reference" "#PWR0121" (id 0) (at 142.24 74.93 0)
+    (property "Reference" "#PWR0138" (id 0) (at 142.24 74.93 0)
       (effects (font (size 1.27 1.27)) hide)
     )
@@
   (symbol (lib_id "Device:R_Small") (at 113.03 92.075 0)
     (in_bom yes) (on_board yes) (fields_autoplaced)
-    (property "Reference" "R11" (id 0) (at 114.935 90.8049 0)
+    (property "Reference" "R8" (id 0) (at 114.935 90.8049 0)
       (effects (font (size 1.27 1.27)) (justify left))
     )
@@
   (symbol (lib_id "Device:R_Small") (at 124.46 74.93 0)
     (in_bom yes) (on_board yes) (fields_autoplaced)
-    (property "Reference" "R12" (id 0) (at 126.365 73.6599 0)
+    (property "Reference" "R9" (id 0) (at 126.365 73.6599 0)
       (effects (font (size 1.27 1.27)) (justify left))
     )
@@
   (symbol (lib_id "power:GND") (at 124.46 100.33 0)
     (in_bom yes) (on_board yes)
-    (property "Reference" "#PWR0116" (id 0) (at 124.46 106.68 0)
+    (property "Reference" "#PWR0137" (id 0) (at 124.46 106.68 0)
       (effects (font (size 1.27 1.27)) hide)
     )
@@
   (symbol (lib_id "Transistor_FET:AO3401A") (at 139.7 78.74 0) (mirror x)
     (in_bom yes) (on_board yes) (fields_autoplaced)
-    (property "Reference" "Q4" (id 0) (at 145.415 77.4699 0)
+    (property "Reference" "Q2" (id 0) (at 145.415 77.4699 0)
       (effects (font (size 1.27 1.27)) (justify left))
     )

Commit message: Start of routing
Parts:
- renumbered Q1 to Q7, Q2 to Q8, R7 to R32, R8 to R33, R9 to R34
Changed lines of the file:
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@@
   (symbol (lib_id "power:+5V") (at 124.46 71.12 0)
     (in_bom yes) (on_board yes)
-    (property "Reference" "#PWR0136" (id 0) (at 124.46 74.93 0)
+    (property "Reference" "#PWR0159" (id 0) (at 124.46 74.93 0)
       (effects (font (size 1.27 1.27)) hide)
     )
@@
   (symbol (lib_id "Device:R_Small") (at 106.045 85.725 90)
     (in_bom yes) (on_board yes) (fields_autoplaced)
-    (property "Reference" "R7" (id 0) (at 106.045 80.01 90))
+    (property "Reference" "R32" (id 0) (at 106.045 80.01 90))
     (property "Value" "100" (id 1) (at 106.045 82.55 90))
     (property "Footprint" "Resistor_SMD:R_0805_2012Metric_Pad1.20x1.40mm_HandSolder" (id 2) (at 106.045 85.725 0)
@@
   (symbol (lib_id "Transistor_FET:AO3400A") (at 121.92 85.725 0)
     (in_bom yes) (on_board yes) (fields_autoplaced)
-    (property "Reference" "Q1" (id 0) (at 128.27 84.4549 0)
+    (property "Reference" "Q7" (id 0) (at 128.27 84.4549 0)
       (effects (font (size 1.27 1.27)) (justify left))
     )
@@
   (symbol (lib_id "power:+5V") (at 142.24 71.12 0)
     (in_bom yes) (on_board yes)
-    (property "Reference" "#PWR0138" (id 0) (at 142.24 74.93 0)
+    (property "Reference" "#PWR0161" (id 0) (at 142.24 74.93 0)
       (effects (font (size 1.27 1.27)) hide)
     )
@@
   (symbol (lib_id "Device:R_Small") (at 113.03 92.075 0)
     (in_bom yes) (on_board yes) (fields_autoplaced)
-    (property "Reference" "R8" (id 0) (at 114.935 90.8049 0)
+    (property "Reference" "R33" (id 0) (at 114.935 90.8049 0)
       (effects (font (size 1.27 1.27)) (justify left))
     )
@@
   (symbol (lib_id "Device:R_Small") (at 124.46 74.93 0)
     (in_bom yes) (on_board yes) (fields_autoplaced)
-    (property "Reference" "R9" (id 0) (at 126.365 73.6599 0)
+    (property "Reference" "R34" (id 0) (at 126.365 73.6599 0)
       (effects (font (size 1.27 1.27)) (justify left))
     )
@@
   (symbol (lib_id "power:GND") (at 124.46 100.33 0)
     (in_bom yes) (on_board yes)
-    (property "Reference" "#PWR0137" (id 0) (at 124.46 106.68 0)
+    (property "Reference" "#PWR0160" (id 0) (at 124.46 106.68 0)
       (effects (font (size 1.27 1.27)) hide)
     )
@@
   (symbol (lib_id "Transistor_FET:AO3401A") (at 139.7 78.74 0) (mirror x)
     (in_bom yes) (on_board yes) (fields_autoplaced)
-    (property "Reference" "Q2" (id 0) (at 145.415 77.4699 0)
+    (property "Reference" "Q8" (id 0) (at 145.415 77.4699 0)
       (effects (font (size 1.27 1.27)) (justify left))
     )

Commit message: more progress, routing almost done
Parts:
- renumbered Q7 to Q3, Q8 to Q4, R32 to R10, R33 to R11, R34 to R12
Changed lines of the file:
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@@
   (symbol (lib_id "power:+5V") (at 124.46 71.12 0)
     (in_bom yes) (on_board yes)
-    (property "Reference" "#PWR0159" (id 0) (at 124.46 74.93 0)
+    (property "Reference" "#PWR0115" (id 0) (at 124.46 74.93 0)
       (effects (font (size 1.27 1.27)) hide)
     )
@@
   (symbol (lib_id "Device:R_Small") (at 106.045 85.725 90)
     (in_bom yes) (on_board yes) (fields_autoplaced)
-    (property "Reference" "R32" (id 0) (at 106.045 80.01 90))
+    (property "Reference" "R10" (id 0) (at 106.045 80.01 90))
     (property "Value" "100" (id 1) (at 106.045 82.55 90))
     (property "Footprint" "Resistor_SMD:R_0805_2012Metric_Pad1.20x1.40mm_HandSolder" (id 2) (at 106.045 85.725 0)
@@
   (symbol (lib_id "Transistor_FET:AO3400A") (at 121.92 85.725 0)
     (in_bom yes) (on_board yes) (fields_autoplaced)
-    (property "Reference" "Q7" (id 0) (at 128.27 84.4549 0)
+    (property "Reference" "Q3" (id 0) (at 128.27 84.4549 0)
       (effects (font (size 1.27 1.27)) (justify left))
     )
@@
   (symbol (lib_id "power:+5V") (at 142.24 71.12 0)
     (in_bom yes) (on_board yes)
-    (property "Reference" "#PWR0161" (id 0) (at 142.24 74.93 0)
+    (property "Reference" "#PWR0121" (id 0) (at 142.24 74.93 0)
       (effects (font (size 1.27 1.27)) hide)
     )
@@
   (symbol (lib_id "Device:R_Small") (at 113.03 92.075 0)
     (in_bom yes) (on_board yes) (fields_autoplaced)
-    (property "Reference" "R33" (id 0) (at 114.935 90.8049 0)
+    (property "Reference" "R11" (id 0) (at 114.935 90.8049 0)
       (effects (font (size 1.27 1.27)) (justify left))
     )
@@
   (symbol (lib_id "Device:R_Small") (at 124.46 74.93 0)
     (in_bom yes) (on_board yes) (fields_autoplaced)
-    (property "Reference" "R34" (id 0) (at 126.365 73.6599 0)
+    (property "Reference" "R12" (id 0) (at 126.365 73.6599 0)
       (effects (font (size 1.27 1.27)) (justify left))
     )
@@
   (symbol (lib_id "power:GND") (at 124.46 100.33 0)
     (in_bom yes) (on_board yes)
-    (property "Reference" "#PWR0160" (id 0) (at 124.46 106.68 0)
+    (property "Reference" "#PWR0116" (id 0) (at 124.46 106.68 0)
       (effects (font (size 1.27 1.27)) hide)
     )
@@
   (symbol (lib_id "Transistor_FET:AO3401A") (at 139.7 78.74 0) (mirror x)
     (in_bom yes) (on_board yes) (fields_autoplaced)
-    (property "Reference" "Q8" (id 0) (at 145.415 77.4699 0)
+    (property "Reference" "Q4" (id 0) (at 145.415 77.4699 0)
       (effects (font (size 1.27 1.27)) (justify left))
     )

Commit message: Exported gerbers and small refinements
Parts:
- renumbered Q3 to Q7, Q4 to Q8, R10 to R32, R11 to R33, R12 to R34
Changed lines of the file:
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@@
   (symbol (lib_id "power:+5V") (at 124.46 71.12 0)
     (in_bom yes) (on_board yes)
-    (property "Reference" "#PWR0115" (id 0) (at 124.46 74.93 0)
+    (property "Reference" "#PWR0159" (id 0) (at 124.46 74.93 0)
       (effects (font (size 1.27 1.27)) hide)
     )
@@
   (symbol (lib_id "Device:R_Small") (at 106.045 85.725 90)
     (in_bom yes) (on_board yes) (fields_autoplaced)
-    (property "Reference" "R10" (id 0) (at 106.045 80.01 90))
+    (property "Reference" "R32" (id 0) (at 106.045 80.01 90))
     (property "Value" "100" (id 1) (at 106.045 82.55 90))
     (property "Footprint" "Resistor_SMD:R_0805_2012Metric_Pad1.20x1.40mm_HandSolder" (id 2) (at 106.045 85.725 0)
@@
   (symbol (lib_id "Transistor_FET:AO3400A") (at 121.92 85.725 0)
     (in_bom yes) (on_board yes) (fields_autoplaced)
-    (property "Reference" "Q3" (id 0) (at 128.27 84.4549 0)
+    (property "Reference" "Q7" (id 0) (at 128.27 84.4549 0)
       (effects (font (size 1.27 1.27)) (justify left))
     )
@@
   (symbol (lib_id "power:+5V") (at 142.24 71.12 0)
     (in_bom yes) (on_board yes)
-    (property "Reference" "#PWR0121" (id 0) (at 142.24 74.93 0)
+    (property "Reference" "#PWR0161" (id 0) (at 142.24 74.93 0)
       (effects (font (size 1.27 1.27)) hide)
     )
@@
   (symbol (lib_id "Device:R_Small") (at 113.03 92.075 0)
     (in_bom yes) (on_board yes) (fields_autoplaced)
-    (property "Reference" "R11" (id 0) (at 114.935 90.8049 0)
+    (property "Reference" "R33" (id 0) (at 114.935 90.8049 0)
       (effects (font (size 1.27 1.27)) (justify left))
     )
@@
   (symbol (lib_id "Device:R_Small") (at 124.46 74.93 0)
     (in_bom yes) (on_board yes) (fields_autoplaced)
-    (property "Reference" "R12" (id 0) (at 126.365 73.6599 0)
+    (property "Reference" "R34" (id 0) (at 126.365 73.6599 0)
       (effects (font (size 1.27 1.27)) (justify left))
     )
@@
   (symbol (lib_id "power:GND") (at 124.46 100.33 0)
     (in_bom yes) (on_board yes)
-    (property "Reference" "#PWR0116" (id 0) (at 124.46 106.68 0)
+    (property "Reference" "#PWR0160" (id 0) (at 124.46 106.68 0)
       (effects (font (size 1.27 1.27)) hide)
     )
@@
   (symbol (lib_id "Transistor_FET:AO3401A") (at 139.7 78.74 0) (mirror x)
     (in_bom yes) (on_board yes) (fields_autoplaced)
-    (property "Reference" "Q4" (id 0) (at 145.415 77.4699 0)
+    (property "Reference" "Q8" (id 0) (at 145.415 77.4699 0)
       (effects (font (size 1.27 1.27)) (justify left))
     )
