File: KiCad/Drawer_Controller_v3/Drawer_Controller/Electrical_Drawer.kicad_sch (KiCad schematic)
At the start: 11 parts, among them U13 TMC2209-LA

Commit message: Finished schematic for electrical drawer
Parts:
- added C47: 4.7uF, symbol Device:C_Polarized_Small
- added D2: white, LED_SMD:LED_0603_1608Metric_Pad1.05x0.95mm_HandSolder, symbol Device:LED_Small
- added R28: 5k, Resistor_SMD:R_0805_2012Metric_Pad1.20x1.40mm_HandSolder, symbol Device:R_Small
- R56: renamed from R50; value 0Ω -> 330mΩ
- R57: renamed from R51; value 0Ω -> 330mΩ
- renumbered C34 to C40, C38 to C41, C35 to C42, C37 to C43, C36 to C44, C39 to C45, R53 to R55, U13 to U14
Connections:
- net DIAG: now also R28.1
- net GND: now also C47.2, D2.1 (K)
- net DAC_Vref: now reaches U14.17 (VREF)
- net at U14.8 (5VOUT): now also C47.1
- new net: D2.2 (A), R28.2
Other:
- note added: "According to the datasheet: 330mΩ resistor results in 0.66A max motor current"
- note added: "Be sure to use a symmetrical sense resistor layout and short and straight sense resistor traces of identical length. Well matching sense resistors ensure best performance. A compact layout with massive ground plane is best to avoid parasitic resistance effects."
- note added: "Datasheet: https://www.trinamic.com/products/integrated-circuits/details/tmc2209-la/"
- note added: "Sense resistors should be carefully selected. The full motor current flows through the sense resistors. Due to chopper operation the sense resistors see pulsed current from the MOSFET bridges. Therefore, a low-inductance type such as film or composition resistors is required to prevent voltage spikes causing ringing on the sense voltage inputs leading to unstable measurement results. Also, a low-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"
- note removed: "Sense resistor connection for coil A and B. Place sense resistor to GND near pin. Tie to GND when using internal sense resistor."
- moved on the sheet: R2, R56, R57
