File: KiCad/Drawer_Controller_v3/Drawer_Controller/Lock_Control.kicad_sch (KiCad schematic)
At the start: 0 parts

Commit message: Starting routing the PCB - WIP
Changed lines of the file:
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@@
     (stroke (width 0) (type default))
   )
-  (wire (pts (xy 163.195 60.325) (xy 168.91 60.325))
+  (wire (pts (xy 163.195 60.325) (xy 194.945 60.325))
     (stroke (width 0) (type default))
   )
@@
     (stroke (width 0) (type default))
   )
-  (wire (pts (xy 163.195 46.355) (xy 168.91 46.355))
+  (wire (pts (xy 163.195 46.355) (xy 194.945 46.355))
     (stroke (width 0) (type default))
   )
-  (wire (pts (xy 154.94 72.39) (xy 168.91 72.39))
+  (wire (pts (xy 154.94 72.39) (xy 194.945 72.39))
     (stroke (width 0) (type default))
   )
@@
     (stroke (width 0) (type default))
   )
+  (label "Lock_VDD_Close" (at 173.99 60.325 0) (fields_autoplaced)
+    (effects (font (size 1.27 1.27)) (justify left bottom))
+  )
+  (label "Switch_Output_Lock" (at 173.355 72.39 0) (fields_autoplaced)
+    (effects (font (size 1.27 1.27)) (justify left bottom))
+  )
+  (label "Lock_VDD_Open" (at 173.355 46.355 0) (fields_autoplaced)
+    (effects (font (size 1.27 1.27)) (justify left bottom))
+  )
   (hierarchical_label "Lock_Close_Control" (shape input) (at 112.395 60.325 180) (fields_autoplaced)
     (effects (font (size 1.27 1.27) bold) (justify right))
   )
-  (hierarchical_label "Lock_VDD_Close" (shape output) (at 168.91 60.325 0) (fields_autoplaced)
+  (hierarchical_label "Lock_VDD_Close" (shape output) (at 194.945 60.325 0) (fields_autoplaced)
     (effects (font (size 1.27 1.27) bold) (justify left))
   )
-  (hierarchical_label "Lock_VDD_Open" (shape output) (at 168.91 46.355 0) (fields_autoplaced)
+  (hierarchical_label "Lock_VDD_Open" (shape output) (at 194.945 46.355 0) (fields_autoplaced)
     (effects (font (size 1.27 1.27) bold) (justify left))
   )
-  (hierarchical_label "Switch_Output_Lock" (shape input) (at 168.91 72.39 0) (fields_autoplaced)
+  (hierarchical_label "Switch_Output_Lock" (shape input) (at 194.945 72.39 0) (fields_autoplaced)
     (effects (font (size 1.27 1.27) bold) (justify left))
   )
