File: KiCad/Partial_Drawer_Controller_v1/Partial_Drawer_Controller_v1/Partial_Drawer_Controller_v1.kicad_pcb (KiCad board)
At the start: 2 copper layers, 408.7 x 50 mm, 642 parts, among them J1 Conn_02x04_Counter_Clockwise, J2 Conn_02x03_Counter_Clockwise, J3 Conn_02x12_Counter_Clockwise, Q1 SS8050, Q10 AO3401A, Q11 AO3400A, Q12 AO3401A, Q13 AO3400A, Q14 AO3401A, Q15 AO3400A, Q16 AO3401A, Q17 AO3400A, Q18 AO3401A, Q19 AO3400A, Q2 2N7002T-7-F, Q20 AO3401A, Q21 AO3400A, Q22 AO3401A, Q23 AO3400A, Q24 AO3401A, Q25 AO3400A, Q26 AO3401A, Q27 AO3400A, Q28 AO3401A, Q29 AO3400A, Q3 2N7002T-7-F, Q30 AO3401A, Q31 AO3400A, Q32 AO3401A, Q33 AO3400A, Q34 AO3401A, Q35 AO3400A, Q36 AO3401A, Q37 AO3400A, Q38 AO3400A, Q39 AO3401A, Q4 AO3400A, Q5 SS8050, Q6 AO3401A, Q7 AO3400A, Q8 AO3401A, Q9 AO3400A, U1 AMS1117-3.3, U11 TMC2209-LA, U13 SN75176BDR, U14 SN75176BDR, U15 SN75176BDR, U19 PCA9535PW,118, U2 LMR33630, U3 PESD2CANFD24L-TR, U4 LP5030RJVR, U5 PCA9535PW,118, U6 CP2102N-Axx-xQFN28, U7 ESP32-WROOM-32E-N8, U8 SN65HVD230, U9 PCA9535PW,118, X1 USB-Micro, X10 Conn_01x03_3.0mm_Molex_Micro_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, X11 Conn_01x03_3.0mm_Molex_Micro_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, X12 Conn_01x03_2.5mm_JST_S04B-XAS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, X13 Conn_01x08_2.5mm_JST_S04B-XAS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, X14 Conn_01x02_2.5mm_JST_S02B-XAS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, X2 Conn_01x04_2.5mm_JST_S04B-XAS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, X3 Conn_01x04_2.5mm_JST_S04B-XAS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, X4 Conn_01x03_3.0mm_Molex_Micro_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, X5 Conn_01x03_3.0mm_Molex_Micro_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, X6 Conn_01x03_3.0mm_Molex_Micro_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, X7 Conn_01x03_3.0mm_Molex_Micro_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, X8 Conn_01x03_3.0mm_Molex_Micro_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, X9 Conn_01x03_3.0mm_Molex_Micro_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

Commit message: feat: adds mounting holes
Parts:
- added H1: MountingHole, MountingHole:MountingHole_3.2mm_M3_DIN965_Pad_TopBottom, F.Cu at (37.5, 39.5)
- added H10: MountingHole, MountingHole:MountingHole_3.2mm_M3_DIN965_Pad_TopBottom, F.Cu at (266.8, 23.7)
- added H11: MountingHole, MountingHole:MountingHole_3.2mm_M3_DIN965_Pad_TopBottom, F.Cu at (292.9, 39.5)
- added H12: MountingHole, MountingHole:MountingHole_3.2mm_M3_DIN965_Pad_TopBottom, F.Cu at (317.9, 23.7)
- added H13: MountingHole, MountingHole:MountingHole_3.2mm_M3_DIN965_Pad_TopBottom, F.Cu at (344.0, 39.5)
- added H14: MountingHole, MountingHole:MountingHole_3.2mm_M3_DIN965_Pad_TopBottom, F.Cu at (368.9, 23.7)
- added H15: MountingHole, MountingHole:MountingHole_3.2mm_M3_DIN965_Pad_TopBottom, F.Cu at (395.1, 39.5)
- added H16: MountingHole, MountingHole:MountingHole_3.2mm_M3_DIN965_Pad_TopBottom, F.Cu at (420.0, 23.7)
- added H17: MountingHole, Robast:MountingHole_4mm_Pad_6.15mm_TopOnly, F.Cu at (31.0, 36.3)
- added H18: MountingHole, Robast:MountingHole_4mm_Pad_6.15mm_TopOnly, F.Cu at (44.0, 36.3)
- added H19: MountingHole, Robast:MountingHole_4mm_Pad_6.15mm_TopOnly, F.Cu at (82.1, 36.3)
- added H2: MountingHole, MountingHole:MountingHole_3.2mm_M3_DIN965_Pad_TopBottom, F.Cu at (62.4, 23.7)
- added H20: MountingHole, Robast:MountingHole_4mm_Pad_6.15mm_TopOnly, F.Cu at (95.1, 36.3)
- added H21: MountingHole, Robast:MountingHole_4mm_Pad_6.15mm_TopOnly, F.Cu at (133.2, 36.3)
- added H22: MountingHole, Robast:MountingHole_4mm_Pad_6.15mm_TopOnly, F.Cu at (146.2, 36.3)
- added H23: MountingHole, Robast:MountingHole_4mm_Pad_6.15mm_TopOnly, F.Cu at (184.2, 36.3)
- added H24: MountingHole, Robast:MountingHole_4mm_Pad_6.15mm_TopOnly, F.Cu at (197.2, 36.3)
- added H25: MountingHole, Robast:MountingHole_4mm_Pad_6.15mm_TopOnly, F.Cu at (235.3, 36.3)
- added H26: MountingHole, Robast:MountingHole_4mm_Pad_6.15mm_TopOnly, F.Cu at (248.3, 36.3)
- added H27: MountingHole, Robast:MountingHole_4mm_Pad_6.15mm_TopOnly, F.Cu at (286.4, 36.3)
- added H28: MountingHole, Robast:MountingHole_4mm_Pad_6.15mm_TopOnly, F.Cu at (299.4, 36.3)
- added H29: MountingHole, Robast:MountingHole_4mm_Pad_6.15mm_TopOnly, F.Cu at (337.5, 36.3)
- added H3: MountingHole, MountingHole:MountingHole_3.2mm_M3_DIN965_Pad_TopBottom, F.Cu at (88.6, 39.5)
- added H30: MountingHole, Robast:MountingHole_4mm_Pad_6.15mm_TopOnly, F.Cu at (350.5, 36.3)
- added H31: MountingHole, Robast:MountingHole_4mm_Pad_6.15mm_TopOnly, F.Cu at (388.6, 36.3)
- added H32: MountingHole, Robast:MountingHole_4mm_Pad_6.15mm_TopOnly, F.Cu at (401.6, 36.3)
- added H33: MountingHole, Robast:MountingHole_3.2mm_M3_Pad_Top_6.4mm_Bottom_9.4mm, F.Cu at (76.8, 59.0)
- added H34: MountingHole, Robast:MountingHole_3.2mm_M3_Pad_Top_6.4mm_Bottom_9.4mm, F.Cu at (127.8, 59.0)
- added H35: MountingHole, Robast:MountingHole_3.2mm_M3_Pad_Top_6.4mm_Bottom_9.4mm, F.Cu at (178.9, 59.0)
- added H36: MountingHole, Robast:MountingHole_3.2mm_M3_Pad_Top_6.4mm_Bottom_9.4mm, F.Cu at (230.0, 59.0)
- added H37: MountingHole, Robast:MountingHole_3.2mm_M3_Pad_Top_6.4mm_Bottom_9.4mm, F.Cu at (281.1, 59.0)
- added H38: MountingHole, Robast:MountingHole_3.2mm_M3_Pad_Top_6.4mm_Bottom_9.4mm, F.Cu at (332.2, 59.0)
- added H39: MountingHole, Robast:MountingHole_3.2mm_M3_Pad_Top_6.4mm_Bottom_9.4mm, F.Cu at (383.3, 59.0)
- added H4: MountingHole, MountingHole:MountingHole_3.2mm_M3_DIN965_Pad_TopBottom, F.Cu at (113.5, 23.7)
- added H40: MountingHole, Robast:MountingHole_3.2mm_M3_Pad_Top_6.4mm_Bottom_9.4mm, F.Cu at (25.7, 59.0)
- added H5: MountingHole, MountingHole:MountingHole_3.2mm_M3_DIN965_Pad_TopBottom, F.Cu at (139.7, 39.5)
- added H6: MountingHole, MountingHole:MountingHole_3.2mm_M3_DIN965_Pad_TopBottom, F.Cu at (164.6, 23.7)
- added H7: MountingHole, MountingHole:MountingHole_3.2mm_M3_DIN965_Pad_TopBottom, F.Cu at (190.7, 39.5)
- added H8: MountingHole, MountingHole:MountingHole_3.2mm_M3_DIN965_Pad_TopBottom, F.Cu at (215.7, 23.7)
- added H9: MountingHole, MountingHole:MountingHole_3.2mm_M3_DIN965_Pad_TopBottom, F.Cu at (241.8, 39.5)
Routing:
- added copper zone on In1.Cu, net GND
- added copper zone on In2.Cu, net GND
Other:
- copper layers 2 -> 4

Commit message: feat: adds some more keepout zones and 3d models for connectors
Parts:
- moved X11 552.0 mm to (412.0, 38.0)
- moved X10 500.7 mm to (361.0, 37.0)
- moved X9 448.3 mm to (309.0, 37.0)
- moved X8 398.1 mm to (259.0, 37.0)
- moved X7 345.9 mm to (207.0, 37.0)
- moved X6 294.9 mm to (156.0, 37.0)
- moved X12 283.7 mm to (165.5, 48.3), turned to -90 degrees
- moved X14 270.9 mm to (165.1, 61.0), turned to -90 degrees
- moved X5 244.1 mm to (105.0, 37.0)
- moved X13 230.2 mm to (111.9, 48.2), turned to -90 degrees
- moved X2 196.9 mm to (68.0, 59.0), turned to -90 degrees
- moved X4 193.6 mm to (54.0, 36.0)
- moved X3 180.2 mm to (68.0, 45.0), turned to -90 degrees

Commit message: feat: first progress in placing parts
Parts:
- D10, D100, D101, D102, D103, D104, D105, D106, D107, D108, D109, D11, D110, D111, D112, D113, D114, D115, D116, D117, D118, D119, D12, D120, D121, D122, D123, D124, D125, D126, D127, D128, D129, D13, D130, D131, D132, D133, D134, D135, D136, D137, D138, D139, D14, D140, D141, D142, D143, D144, D145, D146, D147, D148, D149, D15, D150, D151, D152, D153, D154, D155, D156, D157, D158, D159, D16, D160, D161, D162, D163, D164, D165, D166, D167, D168, D169, D17, D170, D171, D172, D173, D174, D175, D176, D177, D178, D179, D18, D180, D181, D182, D183, D184, D185, D186, D187, D188, D189, D19, D190, D191, D192, D193, D194, D195, D20, D21, D22, D23, D24, D25, D26, D27, D28, D29, D3, D30, D31, D32, D33, D34, D35, D36, D37, D38, D39, D4, D40, D41, D42, D43, D44, D45, D46, D47, D48, D49, D5, D50, D51, D52, D53, D54, D55, D56, D57, D58, D59, D6, D60, D61, D62, D63, D64, D65, D66, D67, D68, D69, D70, D71, D72, D73, D74, D75, D76, D77, D78, D79, D8, D80, D81, D82, D83, D84, D85, D86, D87, D88, D89, D9, D90, D91, D92, D93, D94, D95, D96, D97, D98, D99, R100, R101, R102, R103, R104, R105, R106, R107, R108, R109, R110, R111, R112, R113, R114, R115, R116, R117, R118, R119, R120, R121, R122, R123, R124, R125, R126, R127, R128, R129, R130, R131, R132, R133, R134, R135, R136, R137, R138, R139, R140, R141, R142, R143, R144, R145, R146, R147, R148, R149, R150, R151, R152, R153, R154, R155, R156, R157, R158, R159, R160, R161, R162, R163, R164, R165, R166, R167, R168, R169, R170, R171, R172, R173, R174, R175, R176, R177, R178, R179, R180, R181, R182, R183, R184, R185, R186, R187, R188, R189, R190, R92, R93, R94, R95, R99: moved to B.Cu
- moved F5 574.6 mm to (432.1, 72.1)
- moved F6 574.6 mm to (432.1, 74.5)
- moved F7 574.6 mm to (432.1, 77.0)
- moved JP1 571.2 mm to (439.2, 62.5)
- moved C26 565.2 mm to (439.8, 84.0)
- moved C29 554.7 mm to (429.1, 84.2)
- moved D7 551.5 mm to (437.2, 55.0)
- moved X1 544.7 mm to (425.8, 55.2), turned to 90 degrees
- moved U6 533.0 mm to (396.1, 79.8)
- moved C25 527.1 mm to (416.5, 82.3)
- moved Q2 527.1 mm to (419.6, 86.4)
- moved Q3 527.1 mm to (419.6, 89.5)
- moved S1 527.1 mm to (410.0, 74.8)
- moved S2 527.1 mm to (410.0, 81.5)
- moved Q1 527.1 mm to (416.7, 73.9)
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Other:
- board text added: "${REFERENCE}"
