File: KiCad/Partial_Drawer_Controller_v1/Partial_Drawer_Controller_v1/Switch_Sensing.kicad_sch (KiCad schematic)
At the start: 5 parts

Commit message: feat: minor adjustments and new export of manufacturing files for `Partial_Drawer_controller_v1`
Parts:
- renumbered C28 to C30, F8 to F6, R28 to R59, R29 to R60, S3 to S4
