File: KiCad/Drawer_Controller_v4/Drawer_Controller_v4/Differential_Line_Receiver.kicad_sch (KiCad schematic)
At the start: 6 parts, among them U13 SN75176BDR, U14 SN75176BDR, U15 SN75176BDR

Commit message: feat: completed `Drawer_Controller_v4`
Parts:
- renumbered C68 to C38, C65 to C39, C66 to C40, U14 to U10, U15 to U11, U13 to U9
Changed lines of the file:
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@@
 		(dnp no)
 		(fields_autoplaced yes)
-		(property "Reference" "#PWR0253"
+		(property "Reference" "#PWR0129"
 			(at 29.845 29.845 0)
 			(effects
@@
 			(project "Drawer_Controller_v4"
 				(path "/57f8c193-fe09-43d3-9441-dbd40881d2aa/1cb20bbd-00b4-431f-ae71-2d0dfae72065"
-					(reference "#PWR0253")
+					(reference "#PWR0129")
 					(unit 1)
 				)
@@
 		(dnp no)
 		(fields_autoplaced yes)
-		(property "Reference" "U13"
+		(property "Reference" "U9"
 			(at 139.7 31.75 0)
 			(effects
@@
 			(project "Drawer_Controller_v4"
 				(path "/57f8c193-fe09-43d3-9441-dbd40881d2aa/1cb20bbd-00b4-431f-ae71-2d0dfae72065"
-					(reference "U13")
+					(reference "U9")
 					(unit 1)
 				)
@@
 		(on_board yes)
 		(dnp no)
-		(property "Reference" "#PWR0257"
+		(property "Reference" "#PWR0135"
 			(at 152.4 85.09 0)
 			(effects
@@
 			(project "Drawer_Controller_v4"
 				(path "/57f8c193-fe09-43d3-9441-dbd40881d2aa/1cb20bbd-00b4-431f-ae71-2d0dfae72065"
-					(reference "#PWR0257")
+					(reference "#PWR0135")
 					(unit 1)
 				)
@@
 		(on_board yes)
 		(dnp no)
-		(property "Reference" "#PWR0260"
+		(property "Reference" "#PWR0133"
 			(at 114.3 109.22 0)
 			(effects
@@
 			(project "Drawer_Controller_v4"
 				(path "/57f8c193-fe09-43d3-9441-dbd40881d2aa/1cb20bbd-00b4-431f-ae71-2d0dfae72065"
-					(reference "#PWR0260")
+					(reference "#PWR0133")
 					(unit 1)
 				)
@@
 		(on_board yes)
 		(dnp no)
-		(property "Reference" "#PWR0258"
+		(property "Reference" "#PWR0139"
 			(at 166.37 67.945 0)
 			(effects
@@
 			(project "Drawer_Controller_v4"
 				(path "/57f8c193-fe09-43d3-9441-dbd40881d2aa/1cb20bbd-00b4-431f-ae71-2d0dfae72065"
-					(reference "#PWR0258")
+					(reference "#PWR0139")
 					(unit 1)
 				)
@@
 		(on_board yes)
 		(dnp no)
-		(property "Reference" "#PWR0255"
+		(property "Reference" "#PWR0131"
 			(at 114.3 55.88 0)
 			(effects
@@
 			(project "Drawer_Controller_v4"
 				(path "/57f8c193-fe09-43d3-9441-dbd40881d2aa/1cb20bbd-00b4-431f-ae71-2d0dfae72065"
-					(reference "#PWR0255")
+					(reference "#PWR0131")
 					(unit 1)
 				)
@@
 		(dnp no)
 		(fields_autoplaced yes)
-		(property "Reference" "U15"
+		(property "Reference" "U11"
 			(at 139.7 85.09 0)
 			(effects
@@
 			(project "Drawer_Controller_v4"
 				(path "/57f8c193-fe09-43d3-9441-dbd40881d2aa/1cb20bbd-00b4-431f-ae71-2d0dfae72065"
-					(reference "U15")
+					(reference "U11")
 					(unit 1)
 				)
@@
 		(on_board yes)
 		(dnp no)
-		(property "Reference" "#PWR0265"
+		(property "Reference" "#PWR0142"
 			(at 166.37 106.68 0)
 			(effects
@@
 			(project "Drawer_Controller_v4"
 				(path "/57f8c193-fe09-43d3-9441-dbd40881d2aa/1cb20bbd-00b4-431f-ae71-2d0dfae72065"
-					(reference "#PWR0265")
+					(reference "#PWR0142")
 					(unit 1)
 				)
@@
 		(on_board yes)
 		(dnp no)
-		(property "Reference" "#PWR0256"
+		(property "Reference" "#PWR0132"
 			(at 114.3 82.55 0)
 			(effects
@@
 			(project "Drawer_Controller_v4"
 				(path "/57f8c193-fe09-43d3-9441-dbd40881d2aa/1cb20bbd-00b4-431f-ae71-2d0dfae72065"
-					(reference "#PWR0256")
+					(reference "#PWR0132")
 					(unit 1)
 				)
@@
 		(on_board yes)
 		(dnp no)
-		(property "Reference" "#PWR0259"
+		(property "Reference" "#PWR0140"
 			(at 166.37 80.01 0)
 			(effects
@@
 			(project "Drawer_Controller_v4"
 				(path "/57f8c193-fe09-43d3-9441-dbd40881d2aa/1cb20bbd-00b4-431f-ae71-2d0dfae72065"
-					(reference "#PWR0259")
+					(reference "#PWR0140")
 					(unit 1)
 				)
@@
 		(on_board yes)
 		(dnp no)
-		(property "Reference" "#PWR0263"
+		(property "Reference" "#PWR0136"
 			(at 152.4 111.76 0)
 			(effects
@@
 			(project "Drawer_Controller_v4"
 				(path "/57f8c193-fe09-43d3-9441-dbd40881d2aa/1cb20bbd-00b4-431f-ae71-2d0dfae72065"
-					(reference "#PWR0263")
+					(reference "#PWR0136")
 					(unit 1)
 				)
@@
 		(on_board yes)
 		(dnp no)
-		(property "Reference" "#PWR0262"
+		(property "Reference" "#PWR0138"
 			(at 166.37 53.34 0)
 			(effects
@@
 			(project "Drawer_Controller_v4"
 				(path "/57f8c193-fe09-43d3-9441-dbd40881d2aa/1cb20bbd-00b4-431f-ae71-2d0dfae72065"
-					(reference "#PWR0262")
+					(reference "#PWR0138")
 					(unit 1)
 				)
@@
 		(dnp no)
 		(fields_autoplaced yes)
-		(property "Reference" "C66"
+		(property "Reference" "C40"
 			(at 170.18 95.2499 0)
 			(effects
@@
 			(project "Drawer_Controller_v4"
 				(path "/57f8c193-fe09-43d3-9441-dbd40881d2aa/1cb20bbd-00b4-431f-ae71-2d0dfae72065"
-					(reference "C66")
+					(reference "C40")
 					(unit 1)
 				)
@@
 		(on_board yes)
 		(dnp no)
-		(property "Reference" "#PWR0267"
+		(property "Reference" "#PWR0134"
 			(at 152.4 58.42 0)
 			(effects
@@
 			(project "Drawer_Controller_v4"
 				(path "/57f8c193-fe09-43d3-9441-dbd40881d2aa/1cb20bbd-00b4-431f-ae71-2d0dfae72065"
-					(reference "#PWR0267")
+					(reference "#PWR0134")
 					(unit 1)
 				)
@@
 		(on_board yes)
 		(dnp no)
-		(property "Reference" "#PWR0264"
+		(property "Reference" "#PWR0141"
 			(at 166.37 94.615 0)
 			(effects
@@
 			(project "Drawer_Controller_v4"
 				(path "/57f8c193-fe09-43d3-9441-dbd40881d2aa/1cb20bbd-00b4-431f-ae71-2d0dfae72065"
-					(reference "#PWR0264")
+					(reference "#PWR0141")
 					(unit 1)
 				)
@@
 		(dnp no)
 		(fields_autoplaced yes)
-		(property "Reference" "C68"
+		(property "Reference" "C38"
 			(at 170.18 41.9099 0)
 			(effects
@@
 			(project "Drawer_Controller_v4"
 				(path "/57f8c193-fe09-43d3-9441-dbd40881d2aa/1cb20bbd-00b4-431f-ae71-2d0dfae72065"
-					(reference "C68")
+					(reference "C38")
 					(unit 1)
 				)
@@
 		(dnp no)
 		(fields_autoplaced yes)
-		(property "Reference" "U14"
+		(property "Reference" "U10"
 			(at 139.7 58.42 0)
 			(effects
@@
 			(project "Drawer_Controller_v4"
 				(path "/57f8c193-fe09-43d3-9441-dbd40881d2aa/1cb20bbd-00b4-431f-ae71-2d0dfae72065"
-					(reference "U14")
+					(reference "U10")
 					(unit 1)
 				)
@@
 		(dnp no)
 		(fields_autoplaced yes)
-		(property "Reference" "C65"
+		(property "Reference" "C39"
 			(at 170.18 68.5799 0)
 			(effects
@@
 			(project "Drawer_Controller_v4"
 				(path "/57f8c193-fe09-43d3-9441-dbd40881d2aa/1cb20bbd-00b4-431f-ae71-2d0dfae72065"
-					(reference "C65")
+					(reference "C39")
 					(unit 1)
 				)
@@
 		(dnp no)
 		(fields_autoplaced yes)
-		(property "Reference" "#PWR0254"
+		(property "Reference" "#PWR0130"
 			(at 29.845 60.325 0)
 			(effects
@@
 			(project "Drawer_Controller_v4"
 				(path "/57f8c193-fe09-43d3-9441-dbd40881d2aa/1cb20bbd-00b4-431f-ae71-2d0dfae72065"
-					(reference "#PWR0254")
+					(reference "#PWR0130")
 					(unit 1)
 				)
@@
 		(on_board yes)
 		(dnp no)
-		(property "Reference" "#PWR0261"
+		(property "Reference" "#PWR0137"
 			(at 166.37 41.275 0)
 			(effects
@@
 			(project "Drawer_Controller_v4"
 				(path "/57f8c193-fe09-43d3-9441-dbd40881d2aa/1cb20bbd-00b4-431f-ae71-2d0dfae72065"
-					(reference "#PWR0261")
-					(unit 1)
-				)
+					(reference "#PWR0137")
+					(unit 1)
+				)
