File: KiCad/Drawer_Controller_v4/Drawer_Controller_v4/Power_Stage.kicad_sch (KiCad schematic)
At the start: 23 parts, among them U1 AMS1117-3.3, U2 LMR33630

Commit message: feat: completed `Drawer_Controller_v4`
Parts:
- renumbered C8 to C10, C12 to C11, C9 to C12, C10 to C13, C1 to C2, C2 to C3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
