File: KiCad/Drawer_Controller_v4/Drawer_Controller_v4/Ext_Switch_Sensing.kicad_sch (KiCad schematic)
At the start: 4 parts

Commit message: feat: completed `Drawer_Controller_v4`
Parts:
- renumbered R36 to R16, R28 to R17
Changed lines of the file:
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@@
 		(dnp no)
 		(fields_autoplaced yes)
-		(property "Reference" "R28"
+		(property "Reference" "R17"
 			(at 153.67 77.4699 0)
 			(effects
@@
 			(project "Drawer_Controller_v4"
 				(path "/57f8c193-fe09-43d3-9441-dbd40881d2aa/43bcf634-e9c3-4351-a59f-ee0dcec3115a/b926a9c7-0ab5-42b5-a6cc-eed2281bf581"
-					(reference "R28")
+					(reference "R17")
 					(unit 1)
 				)
 				(path "/57f8c193-fe09-43d3-9441-dbd40881d2aa/289ed4a0-c0fb-403f-8449-e46a308dbcad"
-					(reference "R38")
+					(reference "R46")
 					(unit 1)
 				)
@@
 				)
 				(path "/57f8c193-fe09-43d3-9441-dbd40881d2aa/289ed4a0-c0fb-403f-8449-e46a308dbcad"
-					(reference "F8")
+					(reference "F7")
 					(unit 1)
 				)
@@
 				)
 				(path "/57f8c193-fe09-43d3-9441-dbd40881d2aa/289ed4a0-c0fb-403f-8449-e46a308dbcad"
-					(reference "C18")
+					(reference "C41")
 					(unit 1)
 				)
@@
 		(on_board yes)
 		(dnp no)
-		(property "Reference" "#PWR032"
+		(property "Reference" "#PWR065"
 			(at 128.27 102.87 0)
 			(effects
@@
 			(project "Drawer_Controller_v4"
 				(path "/57f8c193-fe09-43d3-9441-dbd40881d2aa/43bcf634-e9c3-4351-a59f-ee0dcec3115a/b926a9c7-0ab5-42b5-a6cc-eed2281bf581"
-					(reference "#PWR032")
+					(reference "#PWR065")
 					(unit 1)
 				)
 				(path "/57f8c193-fe09-43d3-9441-dbd40881d2aa/289ed4a0-c0fb-403f-8449-e46a308dbcad"
-					(reference "#PWR0103")
+					(reference "#PWR0143")
 					(unit 1)
 				)
@@
 		(dnp no)
 		(fields_autoplaced yes)
-		(property "Reference" "R36"
+		(property "Reference" "R16"
 			(at 139.7 78.74 90)
 			(effects
@@
 			(project "Drawer_Controller_v4"
 				(path "/57f8c193-fe09-43d3-9441-dbd40881d2aa/43bcf634-e9c3-4351-a59f-ee0dcec3115a/b926a9c7-0ab5-42b5-a6cc-eed2281bf581"
-					(reference "R36")
+					(reference "R16")
 					(unit 1)
 				)
 				(path "/57f8c193-fe09-43d3-9441-dbd40881d2aa/289ed4a0-c0fb-403f-8449-e46a308dbcad"
-					(reference "R37")
+					(reference "R45")
 					(unit 1)
 				)
@@
 		(on_board yes)
 		(dnp no)
-		(property "Reference" "#PWR039"
+		(property "Reference" "#PWR067"
 			(at 157.48 102.87 0)
 			(effects
@@
 			(project "Drawer_Controller_v4"
 				(path "/57f8c193-fe09-43d3-9441-dbd40881d2aa/43bcf634-e9c3-4351-a59f-ee0dcec3115a/b926a9c7-0ab5-42b5-a6cc-eed2281bf581"
-					(reference "#PWR039")
+					(reference "#PWR067")
 					(unit 1)
 				)
 				(path "/57f8c193-fe09-43d3-9441-dbd40881d2aa/289ed4a0-c0fb-403f-8449-e46a308dbcad"
-					(reference "#PWR0102")
+					(reference "#PWR0145")
 					(unit 1)
 				)
@@
 		(on_board yes)
 		(dnp no)
-		(property "Reference" "#PWR034"
+		(property "Reference" "#PWR066"
 			(at 151.13 77.47 0)
 			(effects
@@
 			(project "Drawer_Controller_v4"
 				(path "/57f8c193-fe09-43d3-9441-dbd40881d2aa/43bcf634-e9c3-4351-a59f-ee0dcec3115a/b926a9c7-0ab5-42b5-a6cc-eed2281bf581"
-					(reference "#PWR034")
+					(reference "#PWR066")
 					(unit 1)
 				)
 				(path "/57f8c193-fe09-43d3-9441-dbd40881d2aa/289ed4a0-c0fb-403f-8449-e46a308dbcad"
-					(reference "#PWR0101")
-					(unit 1)
-				)
+					(reference "#PWR0144")
+					(unit 1)
+				)
