File: KiCad/Partial_Drawer_Controller_v1_hotfix/Partial_Drawer_Controller_v1_hotfix/Port_Expander.kicad_sch (KiCad schematic)
At the start: 3 parts, among them U8 PCA9535PW,118

Commit message: chore: updates parts and BOM export for `Partial_Drawer_Controller_v1_hotfix`
Parts:
- C53: path_to_docs (none) -> Passive_Components/Capacitors/MLCC/Samsung_Electro-Mechanics
- R201: path_to_docs (none) -> Passive_Components/Resistors/UNI-ROYAL
- U8: path_to_docs (none) -> Semiconductors/Interface_ICs/IO-Expander/NXP
Changed lines of the file:
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@@
 			)
 		)
-		(property "Description" ""
+		(property "Description" "Power symbol creates a global label with name \"+3V3\""
 			(at 114.3 49.53 0)
 			(effects
@@
 			)
 		)
-		(property "Description" ""
+		(property "Description" "Power symbol creates a global label with name \"GND\" , ground"
 			(at 114.3 57.15 0)
 			(effects
@@
 			)
 		)
-		(property "Datasheet" "https://wmsc.lcsc.com/wmsc/upload/file/pdf/v2/lcsc/2304140030_NXP-Semicon-PCA9535PW-118_C255606.pdf"
+		(property "Datasheet" "https://www.nxp.com/docs/en/data-sheet/PCA9535_PCA9535C.pdf"
 			(at 147.32 82.55 0)
 			(effects
@@
 		)
 		(property "OC_RS" ""
+			(at 147.32 82.55 0)
+			(effects
+				(font
+					(size 1.27 1.27)
+				)
+				(hide yes)
+			)
+		)
+		(property "path_to_docs" "Semiconductors/Interface_ICs/IO-Expander/NXP"
 			(at 147.32 82.55 0)
 			(effects
@@
 			)
 		)
+		(property "OC_CONRAD" ""
+			(at 165.1 57.15 0)
+			(effects
+				(font
+					(size 1.27 1.27)
+				)
+				(hide yes)
+			)
+		)
+		(property "OC_RS" ""
+			(at 165.1 57.15 0)
+			(effects
+				(font
+					(size 1.27 1.27)
+				)
+				(hide yes)
+			)
+		)
+		(property "path_to_docs" "Passive_Components/Resistors/UNI-ROYAL"
+			(at 165.1 57.15 0)
+			(effects
+				(font
+					(size 1.27 1.27)
+				)
+				(hide yes)
+			)
+		)
 		(pin "1"
 		)
@@
 			)
 		)
+		(property "OC_CONRAD" ""
+			(at 114.3 53.34 0)
+			(effects
+				(font
+					(size 1.27 1.27)
+				)
+				(hide yes)
+			)
+		)
+		(property "OC_RS" ""
+			(at 114.3 53.34 0)
+			(effects
+				(font
+					(size 1.27 1.27)
+				)
+				(hide yes)
+			)
+		)
+		(property "path_to_docs" "Passive_Components/Capacitors/MLCC/Samsung_Electro-Mechanics"
+			(at 114.3 53.34 0)
+			(effects
+				(font
+					(size 1.27 1.27)
+				)
+				(hide yes)
+			)
+		)
 		(pin "1"
 		)
@@
 			)
 		)
-		(property "Description" ""
+		(property "Description" "Power symbol creates a global label with name \"GND\" , ground"
 			(at 29.21 45.72 0)
 			(effects
@@
 			)
 		)
-		(property "Description" ""
+		(property "Description" "Power symbol creates a global label with name \"+3V3\""
 			(at 29.21 24.13 0)
 			(effects
@@
 			)
 		)
-		(property "Description" ""
+		(property "Description" "Power symbol creates a global label with name \"+3V3\""
 			(at 165.1 50.8 0)
 			(effects
@@
 			)
 		)
-		(property "Description" ""
+		(property "Description" "Power symbol creates a global label with name \"GND\" , ground"
 			(at 127 110.49 0)
 			(effects
