File: KiCad/Drawer_Controller_Distribution_v1_hotfix/Drawer_Controller_Distribution_v1_hotfix/Drawer_Controller_Distribution_v1_hotfix.kicad_sch (KiCad schematic)
At the start: 42 parts, among them J1 RJ45 (6339160-1), J10 Conn_01x02_RS_PRO_3.5mm, J11 Conn_01x02_RS_PRO_3.5mm, J12 Conn_01x02_RS_PRO_3.5mm, J13 Conn_01x02_RS_PRO_3.5mm, J14 Conn_02x05_Odd_Even_Female, J15 Conn_02x05_Odd_Even_Male, J16 Conn_01x02_RS_PRO_3.5mm, J17 Conn_01x02_RS_PRO_3.5mm, J18 Conn_01x02_RS_PRO_3.5mm, J19 Conn_01x02_RS_PRO_3.5mm, J2 RJ45 (6339160-1), J20 Conn_01x02_RS_PRO_3.5mm, J21 Conn_01x02_RS_PRO_3.5mm, J3 RJ45 (6339160-1), J4 RJ45 (6339160-1), J5 Conn_01x02_RS_PRO_5.08mm, J6 Conn_01x03_RS_PRO_3.5mm, J7 Conn_01x02_RS_PRO_5.08mm, J8 Conn_01x02_RS_PRO_3.5mm, J9 Conn_01x02_RS_PRO_3.5mm

Commit message: feat: finished `Drawer_Controller_Distribution_v1_hotfix`
Parts:
- removed F1, F2, F3, F4: RS Pro Fuse Holder (2A), Robast_Footprints:Fuse_Holder_RS_Pro_188-4477, symbol Device:Fuse_Small
- removed F10, F11, F12, F7, F8, F9: RS Pro Fuse Holder, Robast_Footprints:Fuse_Holder_RS_Pro_188-4477, symbol Device:Fuse_Small
- removed F5, F6: Auto_Fuse_Holder, Robast:Fuse_Holder_RS_Pro_188-4477, symbol _Fuse:Auto_Fuse_Holder
- removed J1, J2, J3, J4: RJ45 (6339160-1), Robast_Footprints:TE_6339160-1, symbol 6339160-1:6339160-1
- removed J10, J11, J12, J13, J16, J17, J18, J19, J20, J21, J8, J9: Conn_01x02_RS_PRO_3.5mm, Connector_Phoenix_MC:PhoenixContact_MC_1,5_2-G-3.5_1x02_P3.50mm_Horizontal, symbol Connector_Generic:Conn_01x02
- removed J14: Conn_02x05_Odd_Even_Female, Connector_PinSocket_2.54mm:PinSocket_2x05_P2.54mm_Horizontal, symbol Connector_Generic:Conn_02x05_Odd_Even
- removed J15: Conn_02x05_Odd_Even_Male, Connector_PinHeader_2.54mm:PinHeader_2x05_P2.54mm_Horizontal, symbol Connector_Generic:Conn_02x05_Odd_Even
- removed J5, J7: Conn_01x02_RS_PRO_5.08mm, Connector_Phoenix_MSTB:PhoenixContact_MSTBA_2,5_2-G-5,08_1x02_P5.08mm_Horizontal, symbol Connector_Generic:Conn_01x02
- removed J6: Conn_01x03_RS_PRO_3.5mm, Connector_Phoenix_MC:PhoenixContact_MC_1,5_3-G-3.5_1x03_P3.50mm_Horizontal, symbol Connector_Generic:Conn_01x03
- removed R1: 120, Resistor_SMD:R_0805_2012Metric, symbol Device:R
- added F1, F10, F11, F12, F2, F3, F4, F5, F7, F8, F9: Automotive_Fuse_Holder (2A), Robast:Fuse_Holder_RS_Pro_188-4477, symbol _Fuse:Automotive_Fuse_Holder
- added F6: Automotive_Fuse_Holder (3A), Robast:Fuse_Holder_RS_Pro_188-4477, symbol _Fuse:Automotive_Fuse_Holder
- added R1: 120, Resistor_SMD:R_0805_2012Metric, symbol _R_0805:120
- added X1, X2, X3, X4: RJ45, Robast:TE_RJ45_6339160-1, symbol _Connector:RJ45
- added X10, X11, X12, X13, X14, X15, X16, X17, X18, X19, X8, X9: Conn_01x02_3.5mm_angled, Connector_Phoenix_MC:PhoenixContact_MC_1,5_2-G-3.5_1x02_P3.50mm_Horizontal, symbol _Connector_Phoenix:Conn_01x02_3.5mm_angled
- added X20, X21: Conn_02x05_P2.54mm_angled, Connector_PinHeader_2.54mm:PinHeader_2x05_P2.54mm_Horizontal, symbol _Connector:Conn_02x05_P2.54mm_angled
- added X5, X6: Conn_01x02_5.08mm_angled, Connector_Phoenix_MSTB:PhoenixContact_MSTBA_2,5_2-G-5,08_1x02_P5.08mm_Horizontal, symbol _Connector_Phoenix:Conn_01x02_5.08mm_angled
- added X7: Conn_01x03_3.5mm_angled, Connector_Phoenix_MC:PhoenixContact_MC_1,5_3-G-3.5_1x03_P3.50mm_Horizontal, symbol _Connector_Phoenix:Conn_01x03_3.5mm_angled
Connections:
- net +12V: now also F10.1, F11.1, F12.1, F6.2, X20.10 (Pin_10), X20.9 (Pin_9), X21.10 (Pin_10), X21.9 (Pin_9)
- net +12V_load: now also F10.2, F11.2, F12.2, X14.2 (Pin_2), X15.2 (Pin_2), X16.2 (Pin_2), X17.2 (Pin_2), X18.2 (Pin_2), X19.2 (Pin_2)
- net +24V: now also F1.2, F2.2, F3.2, F4.2, F5.2, F7.1, F8.1, F9.1, X20.1 (Pin_1), X20.2 (Pin_2), X21.1 (Pin_1), X21.2 (Pin_2)
- net +24V-Bus: now also F1.1, F2.1, F3.1, F4.1, X1.1, X1.2, X1.8, X2.1, X2.2, X2.8, X3.1, X3.2, X3.8, X4.1, X4.2, X4.8
- net +24V_load: now also F7.2, F8.2, F9.2, X10.2 (Pin_2), X11.2 (Pin_2), X12.2 (Pin_2), X13.2 (Pin_2), X8.2 (Pin_2), X9.2 (Pin_2)
- net 12V Source: now also F6.1, X6.1 (Pin_1)
- net 24V Source: now also F5.1, X5.2 (Pin_2)
- net CAN+: now also R1.1, X1.4, X2.4, X20.7 (Pin_7), X21.7 (Pin_7), X3.4, X4.4, X7.2 (Pin_2)
- net CAN-: now also R1.2, X1.5, X2.5, X20.5 (Pin_5), X21.5 (Pin_5), X3.5, X4.5, X7.3 (Pin_3)
- net GND: now also X1.3, X1.6, X1.7, X1.SH, X10.1 (Pin_1), X11.1 (Pin_1), X12.1 (Pin_1), X13.1 (Pin_1), X14.1 (Pin_1), X15.1 (Pin_1), X16.1 (Pin_1), X17.1 (Pin_1), X18.1 (Pin_1), X19.1 (Pin_1), X2.3, X2.6, X2.7, X2.SH, X20.3 (Pin_3), X20.4 (Pin_4), X20.6 (Pin_6), X20.8 (Pin_8), X21.3 (Pin_3), X21.4 (Pin_4), X21.6 (Pin_6), X21.8 (Pin_8), X3.3, X3.6, X3.7, X3.SH, X4.3, X4.6, X4.7, X4.SH, X5.1 (Pin_1), X6.2 (Pin_2), X7.1 (Pin_1), X8.1 (Pin_1), X9.1 (Pin_1)
