File: KiCad/Drawer_Controller_v4_hotfix/Drawer_Controller_v4_hotfix/CAN_Communication.kicad_sch (KiCad schematic)
At the start: 13 parts, among them Q1 AO3400A, U4 SN65HVD230

Commit message: feat: updates `Drawer_Controller_v4_hotfix` and `Partial_Drawer_Controller_v1_hotfix` with docs for MOSFETS
Parts:
- Q1: path_to_docs (none) -> Semiconductors/Discrete_Semiconductors/Transistors/MOSFETs/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
Changed lines of the file:
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@@
+			)
+		)
+		(property "OC_CONRAD" ""
+			(at 109.22 118.11 0)
+			(effects
+				(font
+					(size 1.27 1.27)
+				)
+				(hide yes)
+			)
+		)
+		(property "OC_RS" ""
+			(at 109.22 118.11 0)
+			(effects
+				(font
+					(size 1.27 1.27)
+				)
+				(hide yes)
+			)
+		)
+		(property "path_to_docs" "Semiconductors/Discrete_Semiconductors/Transistors/MOSFETs/AO3400A"
+			(at 109.22 118.11 0)
+			(effects
+				(font
+					(size 1.27 1.27)
+				)
+				(hide yes)
 			)
 		)
