File: KiCad/Drawer_Controller_v4_hotfix/Drawer_Controller_v4_hotfix/ESP32_WROOM_32.kicad_sch (KiCad schematic)
At the start: 38 parts, among them Q6 SS8050, Q7 SS8050, Q8 2N7002T-7-F, Q9 2N7002T-7-F, U5 CP2102N-A02-GQFN28R, U6 ESP32-WROOM-32E-N8, X7 USB-Micro

Commit message: feat: updates `Drawer_Controller_v4_hotfix` and `Partial_Drawer_Controller_v1_hotfix` with newest docs
Parts:
- C24: path_to_docs (none) -> Passive_Components/Capacitors/MLCC/FH
Changed lines of the file:
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@@
 			)
 		)
-		(property "Datasheet" "~"
+		(property "Datasheet" "https://www.lcsc.com/datasheet/lcsc_datasheet_2304140030_FH--Guangdong-Fenghua-Advanced-Tech-1206B475K500NT_C29823.pdf"
 			(at 98.425 122.555 0)
 			(effects
@@
 			(at 98.425 122.555 0)
 			(effects
+				(font
+					(size 1.27 1.27)
+				)
+				(hide yes)
+			)
+		)
+		(property "OC_CONRAD" ""
+			(at 98.425 122.555 0)
+			(effects
+				(font
+					(size 1.27 1.27)
+				)
+				(hide yes)
+			)
+		)
+		(property "OC_RS" ""
+			(at 98.425 122.555 0)
+			(effects
+				(font
+					(size 1.27 1.27)
+				)
+				(hide yes)
+			)
+		)
+		(property "path_to_docs" "Passive_Components/Capacitors/MLCC/FH"
+			(at 98.425 122.555 0)
+			(effects

Commit message: feat: updates `Drawer_Controller_v4_hotfix` and `Partial_Drawer_Controller_v1_hotfix` with docs for tactile switch
Parts:
- S2, S3: path_to_docs (none) -> Electromechanical/Switches/Tactile_Switches/TS-1187A-B-A-B
Changed lines of the file:
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@@
+			)
+		)
+		(property "OC_CONRAD" ""
+			(at 95.885 25.4 0)
+			(effects
+				(font
+					(size 1.27 1.27)
+				)
+				(hide yes)
+			)
+		)
+		(property "OC_RS" ""
+			(at 95.885 25.4 0)
+			(effects
+				(font
+					(size 1.27 1.27)
+				)
+				(hide yes)
+			)
+		)
+		(property "path_to_docs" "Electromechanical/Switches/Tactile_Switches/TS-1187A-B-A-B"
+			(at 95.885 25.4 0)
+			(effects
+				(font
+					(size 1.27 1.27)
+				)
+				(hide yes)
 			)
 		)
@@
 			(at 59.055 25.4 0)
 			(effects
+				(font
+					(size 1.27 1.27)
+				)
+				(hide yes)
+			)
+		)
+		(property "OC_CONRAD" ""
+			(at 59.055 25.4 0)
+			(effects
+				(font
+					(size 1.27 1.27)
+				)
+				(hide yes)
+			)
+		)
+		(property "OC_RS" ""
+			(at 59.055 25.4 0)
+			(effects
+				(font
+					(size 1.27 1.27)
+				)
+				(hide yes)
+			)
+		)
+		(property "path_to_docs" "Electromechanical/Switches/Tactile_Switches/TS-1187A-B-A-B"
+			(at 59.055 25.4 0)
+			(effects
