File: KiCad/Drawer_Controller_v4_hotfix/Drawer_Controller_v4_hotfix/VDD_Switch.kicad_sch (KiCad schematic)
At the start: 6 parts, among them Q4 AO3400A, Q5 AO3401A

Commit message: feat: updates `Drawer_Controller_v4_hotfix` and `Partial_Drawer_Controller_v1_hotfix` with docs for MOSFETS
Parts:
- Q4, Q5: path_to_docs (none) -> Semiconductors/Discrete_Semiconductors/Transistors/MOSFETs/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
Changed lines of the file:
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@@
+			)
+		)
+		(property "OC_CONRAD" ""
+			(at 133.35 85.09 0)
+			(effects
+				(font
+					(size 1.27 1.27)
+				)
+				(hide yes)
+			)
+		)
+		(property "OC_RS" ""
+			(at 133.35 85.09 0)
+			(effects
+				(font
+					(size 1.27 1.27)
+				)
+				(hide yes)
+			)
+		)
+		(property "path_to_docs" "Semiconductors/Discrete_Semiconductors/Transistors/MOSFETs/AO3400A"
+			(at 133.35 85.09 0)
+			(effects
+				(font
+					(size 1.27 1.27)
+				)
+				(hide yes)
 			)
 		)
@@
 			(at 151.13 78.74 0)
 			(effects
+				(font
+					(size 1.27 1.27)
+				)
+				(hide yes)
+			)
+		)
+		(property "OC_CONRAD" ""
+			(at 151.13 78.74 0)
+			(effects
+				(font
+					(size 1.27 1.27)
+				)
+				(hide yes)
+			)
+		)
+		(property "OC_RS" ""
+			(at 151.13 78.74 0)
+			(effects
+				(font
+					(size 1.27 1.27)
+				)
+				(hide yes)
+			)
+		)
+		(property "path_to_docs" "Semiconductors/Discrete_Semiconductors/Transistors/MOSFETs/AO3401A"
+			(at 151.13 78.74 0)
+			(effects
